Commit message: Added kinect sensor into the gazebo model

File: simulation/rmc_simulation/robots/rmc_simulation.URDF (robot description, URDF)
Before this commit: robot rmc_simulation, 16 links, 15 joints
Links:
- removed link left_back_wheel_link
- removed link left_bot_back_link
- removed link left_bot_front_link
- removed link left_bot_link
- removed link left_front_wheel_link
- removed link left_mid_wheel_link
- removed link left_top_link
- removed link rear_rocker_link
- removed link right_back_wheel_link
- removed link right_bot_back_link
- removed link right_bot_front_link
- removed link right_bot_link
- removed link right_front_wheel_link
- removed link right_mid_wheel_link
- removed link right_top_link
- added link bl_wheel_link, mass 0.687645998581504; collision mesh filename=package://rmc_simulation/meshes/bl_wheel_link.STL; visual mesh filename=package://rmc_simulation/meshes/bl_wheel_link.STL
- added link br_wheel_link, mass 0.687645998094418; collision mesh filename=package://rmc_simulation/meshes/br_wheel_link.STL; visual mesh filename=package://rmc_simulation/meshes/br_wheel_link.STL
- added link fl_wheel_link, mass 0.687645998625407; collision mesh filename=package://rmc_simulation/meshes/fl_wheel_link.STL; visual mesh filename=package://rmc_simulation/meshes/fl_wheel_link.STL
- added link fr_wheel_link, mass 0.687645998614542; collision mesh filename=package://rmc_simulation/meshes/fr_wheel_link.STL; visual mesh filename=package://rmc_simulation/meshes/fr_wheel_link.STL
- added link ml_wheel_link, mass 0.687645998625407; collision mesh filename=package://rmc_simulation/meshes/ml_wheel_link.STL; visual mesh filename=package://rmc_simulation/meshes/ml_wheel_link.STL
- added link mr_wheel_link, mass 0.687645998625396; collision mesh filename=package://rmc_simulation/meshes/mr_wheel_link.STL; visual mesh filename=package://rmc_simulation/meshes/mr_wheel_link.STL
- link base_link: mass 2.92938025647035 -> 5.21776221348033
Joints:
- removed joint left_back_wheel_joint
- removed joint left_bot_back_joint
- removed joint left_bot_front_joiny
- removed joint left_bot_joint
- removed joint left_front_wheel_joint
- removed joint left_mid_wheel_joint
- removed joint left_top_joint
- removed joint rear_rocker_joint
- removed joint right_back_wheel_joint
- removed joint right_bot_back_link
- removed joint right_bot_front_joint
- removed joint right_bot_joint
- removed joint right_front_wheel_joint
- removed joint right_mid_wheel_link
- removed joint right_top_joint
- added joint bl_wheel_joint: type continuous, parent base_link, child bl_wheel_link, origin xyz=-0.180876313928926 -0.770124006916524 0.0791455484611853 rpy=-1.57079632679488 1.56583942443656 -3.14159265358978, axis 0 -1 0
- added joint br_wheel_joint: type continuous, parent base_link, child br_wheel_link, origin xyz=0.323202134134549 -0.770124006916524 0.07664686034817 rpy=3.13028479554889 -1.11701573915485 -1.56063278319395, axis 0 1 0
- added joint fl_wheel_joint: type continuous, parent base_link, child fl_wheel_link, origin xyz=-0.179281808625283 -0.0779740069165238 0.0778309873766015 rpy=1.5707963267949 1.5707963267949 0, axis 0 -1 0
- added joint fr_wheel_joint: type continuous, parent base_link, child fr_wheel_link, origin xyz=0.322993191374717 -0.0779327659083641 0.0778552780598406 rpy=3.14159265358979 -1.56862653893506 -1.5707963267949, axis 0 1 0
- added joint ml_wheel_joint: type continuous, parent base_link, child ml_wheel_link, origin xyz=-0.179281808625283 -0.433574006916524 0.0778309873766015 rpy=1.5707963267949 1.5707963267949 0, axis 0 -1 0
- added joint mr_wheel_joint: type continuous, parent base_link, child mr_wheel_link, origin xyz=0.322993191374717 -0.433641505259442 0.0778067127306861 rpy=1.5707963267949 -1.5707963267949 0, axis 0 1 0
